File: OriginalData_KiCad/Geekble_Nano_ESP32S3_Ver.2.0/Geekble_Nano_ESP32S3.kicad_pcb (KiCad board)
At the start: 4 copper layers, 43.2 x 17.8 mm, 96 parts, among them J1 USB_C_Receptacle_USB2.0_DIP, SW1 TS-1088-AR02016, SW2 TS-1088-AR02016, U1 ME6217C33M5G, U2 ESP32-S3FH4R2, U3 TPS63070RNMR, Y1 40MHz

Commit message: 2.0
2.0
Parts:
- removed C17: 22uF,16V,0603, Capacitors:C_0603
- removed R12: 680KR,1%, Resistors:R_0402
- removed R13: 130KR,1%, Resistors:R_0402
- C18: value 10uF,6.3V -> 47uF,6.3V,0805; footprint Capacitors:C_0402 -> Capacitors:C_0805
- C19: value 47uF,6.3V,0805 -> 47uF,10V,0805
- C5: value 10uF,6.3V -> 10uF,10V
- U3: value TPS63070RNMR -> TPS630701RNMR
- moved C4 5.58 mm to (45.1, 41.3)
- moved C8 1.20 mm to (39.9, 38.3)
- moved C18 1.04 mm to (47.2, 36.7)
- moved U1 1.04 mm to (43.8, 33.2), turned to 180 degrees
- moved L3 0.80 mm to (40.5, 33.9)
- moved C3 0.76 mm to (45.8, 39.8), turned to 0 degrees
- moved C16 0.75 mm to (40.6, 36.0)
- moved R3 0.62 mm to (38.4, 37.2)
- moved C5 0.56 mm to (45.5, 37.8), turned to 90 degrees
- moved D1 0.25 mm to (38.5, 34.0)
Connections:
- U3 pad 5: Net-(U3-FB) -> +5V
Routing:
- net +3V3: track 52.5 -> 83.0 mm, vias 11 -> 10
- net +5V: track 37.8 -> 42.9 mm, vias 3 -> 2
- net GND: track 51.8 -> 49.0 mm
- net Net-(U3-FB): track 2.55 -> 0.00 mm
- net Net-(C16-Pad2): track 12.4 -> 9.96 mm, vias 1 -> 0
- net VIN: track 54.4 -> 53.0 mm, vias 2 -> 1
- net /B1: track 48.9 -> 47.7 mm
- net Net-(U3-L2): track 6.83 -> 7.81 mm
- net /A4: track 24.0 -> 23.1 mm
- net /A3: track 28.6 -> 27.8 mm
- net Net-(U3-L1): track 5.17 -> 5.92 mm
- net Net-(J1-CC1): track 2.36 -> 2.98 mm
- net /CHIP_PU: track 43.1 -> 42.6 mm
- net /D9: track 17.3 -> 17.1 mm, vias 1 -> 0
- added copper zone on In2.Cu, net GND
- removed copper zone on In2.Cu, net +3V3

Commit message: 2.0
2.0
Parts:
- added C18: 22uF,6.3V,0603, Capacitors:C_0603, F.Cu at (46.9, 37.4)
- C19: renamed from C18; value 47uF,6.3V,0805 -> 22uF,6.3V,0603; footprint Capacitors:C_0805 -> Capacitors:C_0603
- moved C19 2.09 mm to (46.9, 34.7)
- moved C17 0.20 mm to (44.4, 35.9)
- renumbered C9 to C10, C10 to C11, C11 to C12, C12 to C13, C13 to C14, C5 to C15, C14 to C16, C19 to C17, C6 to C5, C16 to C6, C15 to C9, H31 to H1, H6 to H10, H7 to H11, H8 to H12, H9 to H13, H10 to H14, H11 to H15, H12 to H16, H13 to H17, H14 to H18, H15 to H19, H32 to H2, H35 to H20, H36 to H21, H37 to H22, H38 to H23, H39 to H24, H16 to H25, H17 to H26, H18 to H27, H19 to H28, H20 to H29, H33 to H3, H21 to H30, H22 to H31, H23 to H32, H24 to H33, H25 to H34, H26 to H35, H27 to H36, H28 to H37, H29 to H38, H30 to H39, H34 to H4, H1 to H5, H2 to H6, H3 to H7, H4 to H8, H5 to H9, R8 to R10, R9 to R11, R10 to R7, R11 to R8, R7 to R9, U3 to U1, U1 to U3
Routing:
- net /A3: track 27.8 -> 31.8 mm
- net /A2: track 29.4 -> 31.5 mm
- net /A4: track 23.1 -> 24.7 mm
- net /A1: track 32.2 -> 33.8 mm
- net Net-(D2-PadA): track 14.5 -> 13.4 mm, vias 1 -> 0
- net Net-(U1-L2): track 7.81 -> 6.87 mm
- net /B1: track 47.7 -> 46.9 mm
- net /D8: track 14.7 -> 14.2 mm
- net +3V3: track 83.0 -> 82.4 mm
- net Net-(U2-XTAL_N): track 7.82 -> 7.32 mm
