File: OriginalData_KiCad/Geekble_Nano_ESP32S3_Ver.2.0/Geekble_Nano_ESP32S3.kicad_sch (KiCad schematic)
At the start: 96 parts, among them J1 USB_C_Receptacle_USB2.0_DIP, SW1 TS-1088-AR02016, SW2 TS-1088-AR02016, U1 ME6217C33M5G, U2 ESP32-S3FH4R2, U3 TPS63070RNMR, Y1 40MHz

Commit message: 2.0
2.0
Parts:
- removed C17: 22uF,16V,0603, Capacitors:C_0603, symbol Capacitors:22uF,16V,0603
- removed R12: 680KR,1%, Resistors:R_0402, symbol Resistors:680KR,1%
- removed R13: 130KR,1%, Resistors:R_0402, symbol Resistors:130KR,1%
- C18: value 10uF,6.3V -> 47uF,6.3V,0805; footprint Capacitors:C_0402 -> Capacitors:C_0805; symbol Capacitors:10uF,6.3V -> Capacitors:47uF,6.3V,0805; LCSC C15525 -> C16780; Library Type Basic -> Extended; Manufacturer Part Number CL05A106MQ5NUNC -> CL21A476MQYNNNE
- C19: value 47uF,6.3V,0805 -> 47uF,10V,0805; symbol Capacitors:47uF,6.3V,0805 -> Capacitors:47uF,10V,0805; LCSC C16780 -> C124129; Manufacturer Samsung Electro-Mechanics -> Murata Electronics; Manufacturer Part Number CL21A476MQYNNNE -> GRM21BR61A476ME15L
- C5: value 10uF,6.3V -> 10uF,10V; symbol Capacitors:10uF,6.3V -> Capacitors:10uF,10V; LCSC C15525 -> C386033; Library Type Basic -> Extended; Manufacturer Samsung Electro-Mechanics -> Taiyo Yuden; Manufacturer Part Number CL05A106MQ5NUNC -> LDK105CBJ106MVLF
- U3: value TPS63070RNMR -> TPS630701RNMR; symbol Power_Management_ICs:TPS63070RNMR -> Power_Management_ICs:TPS630701RNMR; LCSC C109322 -> C2876599; Manufacturer Part Number TPS63070RNMR -> TPS630701RNMR
Connections:
- net +5V: now also U3.5 (FB)

Commit message: 2.0
2.0
Parts:
- added C18: 22uF,6.3V,0603, Capacitors:C_0603, symbol Capacitors:22uF,6.3V,0603
- C19: renamed from C18; value 47uF,6.3V,0805 -> 22uF,6.3V,0603; footprint Capacitors:C_0805 -> Capacitors:C_0603; symbol Capacitors:47uF,6.3V,0805 -> Capacitors:22uF,6.3V,0603; LCSC C16780 -> C59461; Library Type Extended -> Basic; Manufacturer Part Number CL21A476MQYNNNE -> CL10A226MQ8NRNC
- renumbered C9 to C10, C10 to C11, C11 to C12, C12 to C13, C13 to C14, C5 to C15, C14 to C16, C19 to C17, C6 to C5, C16 to C6, C15 to C9, H31 to H1, H6 to H10, H7 to H11, H8 to H12, H9 to H13, H10 to H14, H11 to H15, H12 to H16, H13 to H17, H14 to H18, H15 to H19, H32 to H2, H35 to H20, H36 to H21, H37 to H22, H38 to H23, H39 to H24, H16 to H25, H17 to H26, H18 to H27, H19 to H28, H20 to H29, H33 to H3, H21 to H30, H22 to H31, H23 to H32, H24 to H33, H25 to H34, H26 to H35, H27 to H36, H28 to H37, H29 to H38, H30 to H39, H34 to H4, H1 to H5, H2 to H6, H3 to H7, H4 to H8, H5 to H9, R8 to R10, R9 to R11, R10 to R7, R11 to R8, R7 to R9, U3 to U1, U1 to U3
Connections:
- net +3V3: now also C18.2
- net GND: now also C18.1
Other:
- moved on the sheet: C19, LED1, R9
